File: userport_expander.kicad_pcb (KiCad board)
At the start: 2 copper layers, 81.1 x 63.1 mm, 21 parts, among them J1 C64-UserPort, U1 16x2_LCD

Commit message: Fixed 4-bit PCB layout, no gerbers yet
Connections:
- U1 pad 10: Net-(D3-Pad2) -> Net-(U1-Pad10)
- U1 pad 11: Net-(U1-Pad11) -> Net-(D0-Pad2)
- U1 pad 12: Net-(U1-Pad12) -> Net-(D1-Pad2)
- U1 pad 13: Net-(U1-Pad13) -> Net-(D2-Pad2)
- U1 pad 14: Net-(U1-Pad14) -> Net-(D3-Pad2)
- U1 pad 7: Net-(D0-Pad2) -> Net-(U1-Pad7)
- U1 pad 8: Net-(D1-Pad2) -> Net-(U1-Pad8)
- U1 pad 9: Net-(D2-Pad2) -> Net-(U1-Pad9)
Routing:
- net Net-(D1-Pad2): track 69.0 -> 63.9 mm
- net Net-(D2-Pad2): track 66.2 -> 61.7 mm
- net Net-(D0-Pad2): track 72.7 -> 68.3 mm, vias 0 -> 1
- net Net-(D3-Pad2): track 62.7 -> 59.6 mm, vias 1 -> 0
- net Net-(D4-Pad2): track 69.6 -> 67.1 mm
- net Net-(RV1-Pad2): track 68.1 -> 69.6 mm
- net GND: vias 0 -> 2
